File: Advanced Flash/genesis_advanced_flash_1-1.kicad_pcb (KiCad board)
At the start: 2 copper layers, 83.8 x 61 mm, 49 parts, among them P1 Genesis Cartridge, SW1 SW_SPDT, U1 29F160, U2 29F160, U3 74LS139, U4 AS6C62256, U5 TPS3613, U6 74HC74, U7 74LS139

Commit message: Add files via upload
Parts:
- added TP3: TPB1,27, Bucketmouse:TestPoint_Pad_D1.0mm, B.Cu at (152.0, 83.0)
- added TP4: TPB1,27, Bucketmouse:TestPoint_Pad_D1.0mm, B.Cu at (148.0, 83.0)
- U3, U7: value 74LS139 -> 74HCT139
- U6: value 74HC74 -> 74HCT74
Routing:
- net +BATT: track 4.17 -> 7.10 mm, vias 0 -> 1
- net Net-(B1-+): track 7.05 -> 9.22 mm, vias 0 -> 1
- net GND: vias 113 -> 114
Other:
- board text added: "R1"
