File: Advanced Flash/genesis_advanced_flash_1-1.kicad_sch (KiCad schematic)
At the start: 46 parts, among them P1 Genesis Cartridge, SW1 SW_SPDT, U1 29F160, U2 29F160, U3 74LS139, U4 AS6C62256, U5 TPS3613, U6 74HC74, U7 74LS139

Commit message: Add files via upload
Parts:
- added TP3, TP4: TPB1,27, Bucketmouse:TestPoint_Pad_D1.0mm, symbol Connector:TestPoint
- U3, U7: value 74LS139 -> 74HCT139
- U6: value 74HC74 -> 74HCT74
- renumbered CB1 to CB, CC1 to CC
Connections:
- net +BATT: now also TP4.1
- net at B1.1 (+), R1.2: now also TP3.1
Other:
- moved on the sheet: R1
Changed lines of the file:
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@@
 	)
 	(junction
+		(at 77.47 91.44)
+		(diameter 0)
+		(color 0 0 0 0)
+	)
+	(junction
 		(at 154.94 21.59)
 		(diameter 0)
@@
 	)
 	(junction
+		(at 95.25 91.44)
+		(diameter 0)
+		(color 0 0 0 0)
+	)
+	(junction
 		(at 26.67 78.74)
 		(diameter 0)
@@
 	(wire
 		(pts
-			(xy 93.98 91.44) (xy 105.41 91.44)
+			(xy 90.17 91.44) (xy 95.25 91.44)
 		)
 		(stroke
@@
 		)
 	)
+	(wire
+		(pts
+			(xy 95.25 91.44) (xy 105.41 91.44)
+		)
+		(stroke
+			(width 0)
+			(type default)
+		)
+	)
 	(bus
 		(pts
@@
 	(wire
 		(pts
-			(xy 77.47 91.44) (xy 86.36 91.44)
+			(xy 77.47 91.44) (xy 82.55 91.44)
 		)
 		(stroke
@@
 	(symbol
 		(lib_id "Device:R")
-		(at 90.17 91.44 270)
+		(at 86.36 91.44 270)
 		(mirror x)
 		(unit 1)
@@
 		(dnp no)
 		(property "Reference" "R1"
-			(at 90.17 86.614 90)
+			(at 86.36 86.614 90)
 			(effects
 				(font
@@
 		)
 		(property "Value" "1k"
-			(at 90.17 88.646 90)
+			(at 86.36 88.646 90)
 			(effects
 				(font
@@
 		)
 		(property "Footprint" "Bucketmouse:R_0603_1608Metric_Boxed"
-			(at 90.17 93.218 90)
+			(at 86.36 93.218 90)
 			(effects
 				(font
@@
 		)
 		(property "Datasheet" "~"
-			(at 90.17 91.44 0)
+			(at 86.36 91.44 0)
 			(effects
 				(font
@@
 		)
 		(property "Description" "Resistor"
-			(at 90.17 91.44 0)
+			(at 86.36 91.44 0)
 			(effects
 				(font
@@
 			)
 		)
-		(property "Value" "74HC74"
+		(property "Value" "74HCT74"
 			(at 89.916 140.208 0)
 			(effects
@@
 			)
 		)
-		(property "Value" "74LS139"
+		(property "Value" "74HCT139"
 			(at 25.4 176.53 90)
 			(effects
@@
 			)
 		)
-		(property "Value" "74HC74"
+		(property "Value" "74HCT74"
 			(at 49.53 180.34 90)
 			(effects
@@
 	)
 	(symbol
+		(lib_id "Connector:TestPoint")
+		(at 95.25 91.44 0)
+		(mirror y)
+		(unit 1)
+		(exclude_from_sim no)
+		(in_bom yes)
+		(on_board yes)
+		(dnp no)
+		(property "Reference" "TP4"
+			(at 95.25 86.106 0)
+			(effects
+				(font
+					(size 1.27 1.27)
+				)
+			)
+		)
+		(property "Value" "TPB1,27"
+			(at 95.25 86.36 0)
+			(effects
+				(font
+					(size 1.27 1.27)
+				)
+				(hide yes)
+			)
+		)
+		(property "Footprint" "Bucketmouse:TestPoint_Pad_D1.0mm"
+			(at 90.17 91.44 0)
+			(effects
+				(font
+					(size 1.27 1.27)
+				)
+				(hide yes)
+			)
+		)
+		(property "Datasheet" "~"
+			(at 90.17 91.44 0)
+			(effects
+				(font
+					(size 1.27 1.27)
+				)
+				(hide yes)
+			)
+		)
+		(property "Description" "test point"
+			(at 95.25 91.44 0)
+			(effects
+				(font
+					(size 1.27 1.27)
+				)
+				(hide yes)
+			)
+		)
+		(pin "1"
+		)
+		(instances
+			(project "genesis_advanced_flash_1-1"
+				(path "/8b2ad2bb-5cbf-4836-a7b2-1cf54b92d388"
+					(reference "TP4")
+					(unit 1)
+				)
+			)
+		)
+	)
+	(symbol
 		(lib_id "Device:R")
 		(at 177.8 138.43 0)
@@
 			)
 		)
-		(property "Value" "74LS139"
+		(property "Value" "74HCT139"
 			(at 177.8 27.94 0)
 			(effects
@@
 			)
 		)
-		(property "Value" "74LS139"
+		(property "Value" "74HCT139"
 			(at 119.38 186.69 0)
 			(effects
@@
 			)
 		)
-		(property "Value" "74LS139"
+		(property "Value" "74HCT139"
 			(at 172.212 96.52 0)
 			(effects
@@
 			)
 		)
-		(property "Value" "74LS139"
+		(property "Value" "74HCT139"
 			(at 177.8 60.96 0)
 			(effects
@@
 		(on_board yes)
 		(dnp no)
-		(property "Reference" "CC1"
+		(property "Reference" "CC"
 			(at 58.928 140.97 0)
 			(effects
@@
 			(project "Genesis_Advanced_1-0"
 				(path "/8b2ad2bb-5cbf-4836-a7b2-1cf54b92d388"
-					(reference "CC1")
+					(reference "CC")
 					(unit 1)
 				)
@@
 			)
 		)
-		(property "Value" "74LS139"
+		(property "Value" "74HCT139"
 			(at 127 159.004 0)
 			(effects
@@
 		(on_board yes)
 		(dnp no)
-		(property "Reference" "CB1"
+		(property "Reference" "CB"
 			(at 135.128 43.18 0)
 			(effects
@@
 			(project "Genesis_Advanced_1-0"
 				(path "/8b2ad2bb-5cbf-4836-a7b2-1cf54b92d388"
-					(reference "CB1")
+					(reference "CB")
 					(unit 1)
 				)
@@
 			)
 		)
-		(property "Value" "74HC74"
+		(property "Value" "74HCT74"
 			(at 34.036 146.558 0)
 			(effects
@@
 					(unit 1)
 				)
+			)
+		)
+	)
+	(symbol
+		(lib_id "Connector:TestPoint")
+		(at 77.47 91.44 0)
+		(mirror y)
+		(unit 1)
+		(exclude_from_sim no)
+		(in_bom yes)
+		(on_board yes)
+		(dnp no)
+		(property "Reference" "TP3"
+			(at 77.47 86.106 0)
+			(effects
+				(font
+					(size 1.27 1.27)
+				)
+			)
+		)
+		(property "Value" "TPB1,27"
+			(at 77.47 86.36 0)
+			(effects
+				(font
+					(size 1.27 1.27)
+				)
+				(hide yes)
+			)
+		)
+		(property "Footprint" "Bucketmouse:TestPoint_Pad_D1.0mm"
+			(at 72.39 91.44 0)
+			(effects
+				(font
+					(size 1.27 1.27)
+				)
+				(hide yes)
+			)
+		)
+		(property "Datasheet" "~"
+			(at 72.39 91.44 0)
+			(effects
+				(font
+					(size 1.27 1.27)
+				)
+				(hide yes)
+			)
+		)
+		(property "Description" "test point"
+			(at 77.47 91.44 0)
+			(effects
+				(font
+					(size 1.27 1.27)
+				)
+				(hide yes)
+			)
+		)
+		(pin "1"
+		)
+		(instances
+			(project "genesis_advanced_flash_1-1"
+				(path "/8b2ad2bb-5cbf-4836-a7b2-1cf54b92d388"
+					(reference "TP3")
+					(unit 1)
+				)
