File: Advanced Flash/genesis_advanced_flash_1-2.kicad_pcb (KiCad board)
At the start: 2 copper layers, 83.8 x 61 mm, 51 parts, among them P1 Genesis Cartridge, SW1 SW_SPDT, U1 29F160, U2 29F160, U3 74HCT139, U4 AS6C62256, U5 TPS3613, U6 74HCT74, U7 74HCT139

Commit message: Add files via upload
Other:
- board text added: "GENESIS/MD/32X FLASH CART PCB"
- board text removed: "GENESIS/MEGA DRIVE FLASH CART PCB"
Changed lines of the file:
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@@
 			(drillshape 0)
 			(scaleselection 1)
-			(outputdirectory "genesis_advanced_flash_1-1_GERBERS/")
+			(outputdirectory "genesis_advanced_flash_1-2_GERBERS/")
 		)
 	)
@@
 		)
 	)
-	(gr_text "GENESIS/MEGA DRIVE FLASH CART PCB"
+	(gr_text "GENESIS/MD/32X FLASH CART PCB"
 		(at 184.7469 131.8514 0)
 		(layer "F.SilkS")
