File: Advanced UV/Genesis_Advanced_1-0.kicad_sch (KiCad schematic)
At the start: 50 parts, among them P1 Genesis Cartridge, Q1A1 2N3904, Q1B1 MMBT3904, U1 27C322, U2 AS6C62256, U3 74HC74, U4 74LS139

Commit message: Add files via upload
Parts:
- U3: value 74HC74 -> 74HCT74
- U4: value 74LS139 -> 74HCT139
- renumbered CB1 to CB, CC1 to CC
Changed lines of the file:
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@@
 			)
 		)
-		(property "Value" "74HC74"
+		(property "Value" "74HCT74"
 			(at 107.696 104.648 0)
 			(effects
@@
 			)
 		)
-		(property "Value" "74LS139"
+		(property "Value" "74HCT139"
 			(at 92.71 176.53 90)
 			(effects
@@
 			)
 		)
-		(property "Value" "74HC74"
+		(property "Value" "74HCT74"
 			(at 116.84 180.34 90)
 			(effects
@@
 			)
 		)
-		(property "Value" "74LS139"
+		(property "Value" "74HCT139"
 			(at 142.24 152.4 0)
 			(effects
@@
 		(on_board yes)
 		(dnp no)
-		(property "Reference" "CC1"
+		(property "Reference" "CC"
 			(at 70.358 140.97 0)
 			(effects
@@
 			(project "Genesis_Advanced_1-0"
 				(path "/8b2ad2bb-5cbf-4836-a7b2-1cf54b92d388"
-					(reference "CC1")
+					(reference "CC")
 					(unit 1)
 				)
@@
 			)
 		)
-		(property "Value" "74LS139"
+		(property "Value" "74HCT139"
 			(at 149.86 124.714 0)
 			(effects
@@
 		(on_board yes)
 		(dnp no)
-		(property "Reference" "CB1"
+		(property "Reference" "CB"
 			(at 163.068 43.18 0)
 			(effects
@@
 			(project "Genesis_Advanced_1-0"
 				(path "/8b2ad2bb-5cbf-4836-a7b2-1cf54b92d388"
-					(reference "CB1")
+					(reference "CB")
 					(unit 1)
 				)
@@
 			)
 		)
-		(property "Value" "74HC74"
+		(property "Value" "74HCT74"
 			(at 152.146 185.928 0)
 			(effects
